File: HARDWARE/ETH1ACPL-C79x/ETH1ACPL-C79x.kicad_pcb (KiCad board)
At the start: 4 copper layers, 100 x 45 mm, 143 parts, among them J201 20021111-00010T4LF, J301 1715721, J401 RJ45_Wuerth_7499010121A, J501 1710072, Q301 SI5618A, Q302 MMBT3904, U201 LT6350xMS8, U202 REF1933AIDDCT, U203 STM32H743VITx, U204 24LC08B-E/MS, U301 TSR_1-2450, U302 TLV62568DBV, U401 LAN8742A, U501 DG412LEDQ, U502 TBA 1-0511HI, U503 ACPL-C79B, U504 DG419LEDY, U505 OPA2340UA, Y201 NX5032GA-16, Y401 NX5032GA-25

Commit message: Development
Parts:
- removed the REF** at (107.6, 116.0)
- C202, C204, C205, C206, C207, C208, C209, C210, C211, C213, C221, C401, C402, C403, C404, C405, C407, C408, C409, C410, C411, C412, D301, R402, R403, R404, R405, R406: moved to B.Cu
- moved C205 201.9 mm to (163.2, 84.8), turned to 90 degrees
- moved C202 199.9 mm to (161.7, 84.8), turned to 90 degrees
- moved C206 199.2 mm to (161.0, 93.6), turned to 90 degrees
- moved C207 199.1 mm to (159.9, 84.8), turned to 90 degrees
- moved C412 197.2 mm to (182.4, 88.1), turned to 90 degrees
- moved C204 196.9 mm to (158.4, 84.8), turned to 90 degrees
- moved C411 193.9 mm to (180.1, 101.2), turned to -90 degrees
- moved C209 193.7 mm to (159.9, 89.3), turned to -90 degrees
- moved C213 192.4 mm to (158.4, 92.7)
- moved C211 192.3 mm to (158.4, 89.3), turned to -90 degrees
- moved C407 191.0 mm to (172.5, 100.8), turned to -90 degrees
- moved C404 190.6 mm to (171.6, 87.6), turned to 90 degrees
- moved C210 189.9 mm to (155.8, 84.8), turned to 90 degrees
- moved C208 188.6 mm to (154.8, 92.7)
- moved C402 187.6 mm to (169.3, 91.6), turned to 90 degrees
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Connections:
- U203 pad 28: unconnected-(U203-PA4-Pad28) -> /MCU/MCU_G100
- U203 pad 29: unconnected-(U203-PA5-Pad29) -> /MCU/MCU_G10
- U203 pad 30: unconnected-(U203-PA6-Pad30) -> /MCU/MCU_G1
- U203 pad 37: /MCU/MCU_G100 -> unconnected-(U203-PE7-Pad37)
- U203 pad 38: /MCU/MCU_G10 -> unconnected-(U203-PE8-Pad38)
- U203 pad 40: /MCU/MCU_G1 -> unconnected-(U203-PE10-Pad40)
Routing:
- net GND1: track 0.00 -> 77.6 mm, vias 0 -> 4
- net +3.3V: track 0.00 -> 71.6 mm, vias 0 -> 26
- net /MCU/NRST: track 0.00 -> 58.3 mm, vias 0 -> 2
- net +1.65V: track 0.00 -> 49.3 mm, vias 0 -> 3
- net VCCQ: track 0.00 -> 38.4 mm, vias 0 -> 4
- net GND: track 0.00 -> 37.6 mm, vias 0 -> 10
- net /Ethernet/RMII_MDIO: track 0.00 -> 34.7 mm, vias 0 -> 2
- net Net-(D501-K-Pad3): track 0.00 -> 30.9 mm, vias 0 -> 3
- net /Ethernet/RMII_TXEN: track 0.00 -> 30.4 mm, vias 0 -> 2
- net /Ethernet/RMII_CRS_DV: track 0.00 -> 30.3 mm, vias 0 -> 2
- net /Ethernet/RMII_MDC: track 0.00 -> 30.3 mm, vias 0 -> 2
- net /Ethernet/RMII_RXD1: track 0.00 -> 30.3 mm, vias 0 -> 2
- net /Ethernet/RMII_RXD0: track 0.00 -> 30.2 mm, vias 0 -> 2
- net /Ethernet/RMII_TXD0: track 0.00 -> 30.2 mm, vias 0 -> 2
- net /Ethernet/RMII_TXD1: track 0.00 -> 30.2 mm, vias 0 -> 2
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- added copper zone on B.Cu, net +1.65V
- added copper zone on B.Cu, net +3.3V
- added copper zone on F.Cu, net +3.3V
- added copper zone on In2.Cu, net +3.3V
- added copper zone on B.Cu, net +3.3VADC
- added copper zone on B.Cu, net +5V
- added copper zone on F.Cu, net +5V
- added copper zone on In2.Cu, net +5V
- added copper zone on B.Cu, net Earth
- added copper zone on F.Cu, net Earth
- added copper zone on B.Cu, net GND
- added copper zone on F.Cu, net GND
- added copper zone on In1.Cu, net GND
- added copper zone on B.Cu, net Net-(D301-K)
- added copper zone on F.Cu, net Net-(D301-K)
- added copper zone on B.Cu, net Net-(J301-Pin_1)
- added copper zone on B.Cu, net Net-(Q301-D)
- added copper zone on F.Cu, net Net-(Q301-D)
- added copper zone on F.Cu, net Net-(U302-SW)
- added copper zone on B.Cu, net VCCQ
- added copper zone on F.Cu, net VCCQ
- added copper zone on In2.Cu, net VCCQ
- added copper zone on B.Cu, net VDDA
Other:
- board text added: "VOLTAGE MEASUREMENT"

Commit message: Development
Parts:
- moved H101 4.00 mm to (123.0, 81.5)
- moved H103 4.00 mm to (123.0, 119.5)
- moved R504 0.13 mm to (108.6, 112.0)
- moved R508 0.13 mm to (108.6, 117.0)
- moved R501 0.13 mm to (106.4, 88.9)
- moved R502 0.13 mm to (108.7, 88.9)
- moved R503 0.13 mm to (106.3, 112.0)
- moved R505 0.13 mm to (106.4, 83.9)
- moved R506 0.13 mm to (108.7, 83.9)
- moved R507 0.13 mm to (106.3, 117.0)
Routing:
- net GND: track 37.6 -> 66.7 mm, vias 10 -> 30
- net GND1: track 77.6 -> 73.7 mm
- net /MCU/VOUT: track 17.8 -> 15.8 mm
- net /Ethernet/LED2: track 15.3 -> 16.4 mm
- net +5V: track 18.5 -> 19.3 mm
- net /MCU/MCU_DEF: track 11.4 -> 10.8 mm
Other:
- outline, holes or cut-outs redrawn

Commit message: Development
Parts:
- added REF**: Symbol_Attention_Triangle_8x7mm_Copper, Symbol:Symbol_Attention_Triangle_8x7mm_Copper, B.Cu at (121.2, 90.7)
- U202: footprint Package_TO_SOT_SMD:TSOT-23-5_HandSoldering -> Package_TO_SOT_SMD:TSOT-23-5
- moved REF** 2.71 mm to (121.2, 90.7)
- moved R501 1.02 mm to (105.4, 88.9)
- moved R502 1.02 mm to (107.7, 88.9)
- moved R503 1.02 mm to (105.3, 112.0)
- moved R505 1.02 mm to (105.4, 83.9)
- moved R506 1.02 mm to (107.7, 83.9)
- moved R507 1.02 mm to (105.3, 117.0)
- moved R504 1.02 mm to (107.6, 112.0)
- moved R508 1.02 mm to (107.6, 117.0)
Routing:
- net GND: track 66.7 -> 69.1 mm, vias 30 -> 31
- net Net-(J501-Pin_2): track 11.2 -> 13.0 mm
- net Net-(J501-Pin_1): track 11.3 -> 13.1 mm
- net +5V: track 19.3 -> 18.2 mm
- net Net-(R507-Pad2): track 9.27 -> 10.4 mm
- net Net-(R505-Pad2): track 9.14 -> 10.3 mm
- net GND1: track 73.7 -> 74.6 mm
- net +1.65V: track 49.3 -> 48.3 mm
- net +3.3VADC: track 16.5 -> 15.7 mm
- net Net-(U503-IN+): track 19.7 -> 19.0 mm
- net Net-(U503-IN-): track 19.7 -> 19.1 mm
- net +5VP: track 24.7 -> 25.3 mm
- net /MCU/VOUT: track 15.8 -> 15.2 mm

Commit message: Development
Parts:
- moved C513 3.86 mm to (121.8, 111.4)
- moved C508 1.58 mm to (121.8, 108.6)
Routing:
- net GND1: track 74.6 -> 73.2 mm
- net +5VP: track 25.3 -> 24.4 mm
Other:
- outline, holes or cut-outs redrawn
- board text added: "ETH1ACPL-C79x V1.00 Default IP : 192.168.1.18"

Commit message: Development
Parts:
- moved H101 19.5 mm to (103.5, 81.5)
- moved H103 19.5 mm to (103.5, 119.5)
- moved C304 10.3 mm to (166.4, 112.8)
- moved C303 10.3 mm to (176.4, 114.9)
- moved REF** 7.62 mm to (117.3, 84.1)
- moved R501 5.54 mm to (103.5, 94.1)
- moved R502 5.54 mm to (105.8, 94.1)
- moved R505 5.54 mm to (103.5, 89.2)
- moved R506 5.54 mm to (105.8, 89.2)
- moved R503 5.50 mm to (103.5, 106.8)
- moved R504 5.50 mm to (105.8, 106.8)
- moved R507 5.50 mm to (103.5, 111.8)
- moved R508 5.50 mm to (105.8, 111.8)
- moved R511 0.99 mm to (114.2, 117.6)
- moved R512 0.99 mm to (116.5, 117.6)
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Routing:
- net Net-(R505-Pad2): track 10.3 -> 15.3 mm
- net Net-(J501-Pin_2): track 13.0 -> 7.97 mm
- net Net-(R507-Pad2): track 10.4 -> 15.4 mm
- net Net-(J501-Pin_1): track 13.1 -> 9.70 mm
- net Net-(D201-BK): track 9.83 -> 10.3 mm
- net Net-(D201-RK): track 9.53 -> 10.0 mm
Other:
- outline, holes or cut-outs redrawn

Commit message: Development
Parts:
- removed REF** (x2): Symbol_Attention_Triangle_8x7mm_Copper, Symbol:Symbol_Attention_Triangle_8x7mm_Copper
- added SYM501: SYM_Flash_Small, ETH1ACPL-C79x:Symbol_Attention_Triangle_8x7mm_Copper, F.Cu at (122.0, 88.4)
- added SYM502: SYM_Flash_Small, ETH1ACPL-C79x:Symbol_Attention_Triangle_8x7mm_Copper, B.Cu at (122.0, 88.4)
- R530: value 100 -> 0
Connections:
- R524 pad 2: GND -> +1.65V
Routing:
- net +1.65V: track 48.3 -> 59.6 mm
- net GND: track 69.5 -> 70.9 mm, vias 31 -> 32
- net Net-(R523-Pad2): track 16.4 -> 15.8 mm
- net /Ethernet/MODE0: track 2.86 -> 3.38 mm
- net +3.3V: vias 26 -> 24

Commit message: PCB design changes.
Parts:
- removed L301: CSHB0415-2R2M, ETH1ACPL-C79x:CSHB0415
- removed R303: 45k3, Resistor_SMD:R_0603_1608Metric_Pad0.98x0.95mm_HandSolder
- removed R304: 10k, Resistor_SMD:R_0603_1608Metric_Pad0.98x0.95mm_HandSolder
- removed the R526 at (140.3, 95.6)
- added C213: DNP, Capacitor_SMD:C_0603_1608Metric_Pad1.08x0.95mm_HandSolder, F.Cu at (155.8, 89.5)
- added FID101: Fiducial, Fiducial:Fiducial_1.5mm_Mask3mm, F.Cu at (108.6, 80.1)
- added FID102: Fiducial, Fiducial:Fiducial_1.5mm_Mask3mm, B.Cu at (108.6, 80.1)
- added FID103: Fiducial, Fiducial:Fiducial_1.5mm_Mask3mm, F.Cu at (190.4, 120.8)
- added FID104: Fiducial, Fiducial:Fiducial_1.5mm_Mask3mm, B.Cu at (190.4, 120.8)
- D201: value ASCB-JTC2-0A308 -> ASMB-MTB1-0B3A2
- RN201: value 680 -> EXB-V8V102JV
- U302: value TLV62568DBV -> LM1117MP-3.3/NOPB; footprint Package_TO_SOT_SMD:SOT-23-5 -> Package_TO_SOT_SMD:SOT-223-3_TabPin2
- moved C304 4.96 mm to (170.2, 116.0), turned to 180 degrees
- moved C305 4.95 mm to (168.3, 101.6), turned to 90 degrees
- moved U302 3.64 mm to (169.4, 109.5), turned to 90 degrees
- moved C210 1.91 mm to (153.9, 84.8)
- moved R204 1.64 mm to (153.3, 90.8)
- moved R203 1.57 mm to (153.3, 88.3)
- moved FB401 0.25 mm to (171.7, 101.3)
- renumbered C213 to C214, C214 to C215, C215 to C216, C216 to C217, C217 to C218, C218 to C219, C219 to C220, C220 to C221, C221 to C222, R207 to R203, R208 to R204, R203 to R205, R204 to R206, R205 to R207, R206 to R208, R527 to R526, R528 to R527, R529 to R528, R530 to R529, U504 to U502, U502 to U503, U503 to U504
Connections:
- C210 pad 1: +3.3V -> +3.3VADC
- U201 pad 3: +3.3V -> +3.3VADC
- U201 pad 7: +3.3V -> +3.3VADC
- U302 pad 1: +5V -> GND
- U302 pad 2: GND -> +3.3V
- U302 pad 3: Net-(U302-SW) -> +5V
Routing:
- net +3.3V: track 71.7 -> 58.7 mm, vias 24 -> 18
- net +3.3VADC: track 15.7 -> 26.2 mm, vias 2 -> 3
- net GND: track 70.9 -> 62.1 mm, vias 32 -> 26
- net Net-(U302-FB): track 4.31 -> 0.00 mm
- net Net-(U201-OUT2): track 8.06 -> 11.7 mm
- net +5V: track 17.9 -> 15.5 mm, vias 7 -> 4
- net /MCU/VOUTN: track 4.72 -> 2.80 mm
- net Net-(U201--IN1): track 8.72 -> 10.4 mm
- net /MCU/VOUTP: track 6.68 -> 5.30 mm
- net /MCU/VOUT: track 15.2 -> 16.1 mm
- net Net-(D501-K-Pad3): track 30.9 -> 30.3 mm, vias 3 -> 2
- removed copper zone on F.Cu, net Net-(U302-SW)

Commit message: Hardware design
Parts:
- added C518: 68p, Capacitor_SMD:C_0603_1608Metric_Pad1.08x0.95mm_HandSolder, B.Cu at (130.1, 125.6)
- added C519: 68p, Capacitor_SMD:C_0603_1608Metric_Pad1.08x0.95mm_HandSolder, B.Cu at (130.1, 128.1)
- added RN501: MPMT50011002AT5, Package_TO_SOT_SMD:SOT-23, B.Cu at (134.7, 126.8)
- added RN502: MPMT50011002AT5, Package_TO_SOT_SMD:SOT-23, B.Cu at (134.7, 131.4)
- R526: value 180k/0.1% -> 180k/0.05%
- R527: value 18k/0.1% -> 18k/0.05%
- R528: value 2k/0.1% -> 2k/0.05%
