File: HARDWARE/ETH1ACPL-C79x/ETH1ACPL-C79x.kicad_pcb (KiCad board)
At the start: 4 copper layers, 100 x 45 mm, 148 parts, among them J201 20021111-00010T4LF, J301 1715721, J401 RJ45_Wuerth_7499010121A, J501 1710072, Q301 SI5618A, Q302 MMBT3904, U201 LT6350xMS8, U202 REF1933AIDDCT, U203 STM32H743VITx, U204 24LC08B-E/MS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

Commit message: Hardware design
Parts:
- U202: footprint Package_TO_SOT_SMD:TSOT-23-5 -> Package_TO_SOT_SMD:SOT-23-5_HandSoldering
- moved C519 33.4 mm to (140.3, 96.4)
- moved RN502 28.8 mm to (135.0, 102.6), turned to -90 degrees
- moved RN501 28.2 mm to (135.0, 98.6), turned to 90 degrees
- moved C518 27.6 mm to (142.1, 100.8), turned to -90 degrees
- moved C507 4.81 mm to (133.7, 94.7), turned to 90 degrees
Routing:
- net (no net): track 0.00 -> 84.3 mm
- net Net-(C518-Pad2): track 15.8 -> 31.2 mm
- net Net-(U505A--): track 10.1 -> 14.6 mm, vias 0 -> 2
- net Net-(U505A-+): track 9.27 -> 12.9 mm, vias 0 -> 2
- net GND: track 62.1 -> 59.4 mm, vias 26 -> 24
- net Net-(U504-OUT-): track 3.26 -> 4.44 mm, vias 0 -> 1
- net Net-(U505B-+): track 18.2 -> 19.3 mm
- net +5V: track 15.5 -> 16.4 mm
- net +1.65V: track 59.4 -> 58.8 mm
- net +3.3V: track 58.7 -> 58.1 mm
- net Net-(U504-OUT+): track 3.26 -> 3.72 mm, vias 0 -> 1
Other:
- board text added: "1"
- board text added: "2"
- board text added: "3"
- board text added: "4"
