File: HARDWARE/ETH1ACPL-C79x/MCU.kicad_sch (KiCad schematic)
At the start: 37 parts, among them J401 20021111-00010T4LF, U203 REF1933AIDDCT, U204 LT6350xMS8, U403 STM32H743VITx, U404 24LC08B-E/MS, Y401 NX5032GA-16

Commit message: Development
Parts:
- added R207, R208: 0, Resistor_SMD:R_0603_1608Metric_Pad0.98x0.95mm_HandSolder, symbol Device:R
- renumbered C206 to C202, C207 to C205, R205 to R201, U204 to U201, U203 to U202
Connections:
- net VOUTN: now also R208.2; no longer U201.5 (OUT2)
- net VOUTP: now also R207.2; no longer R201.2, U201.1 (-IN1), U201.4 (OUT1)
- net MCU_DIV1: no longer names the net of U403.45 (PE15)
- net MCU_DIV10: no longer names the net of U403.41 (PE11)
- net MCU_DIV100: no longer names the net of U403.42 (PE12)
- net MCU_DIV_ENA: no longer names the net of U403.44 (PE14)
- net MCU_MEAS_ENA: no longer names the net of U403.39 (PE9)
- new net: R201.2, R207.1, U201.1 (-IN1), U201.4 (OUT1)
- new net: R208.1, U201.5 (OUT2)
- no-connect marks 57 -> 62

Commit message: Development
Connections:
- net MCU_G1: now also U403.30 (PA6); no longer U403.40 (PE10)
- net MCU_G10: now also U403.29 (PA5); no longer U403.38 (PE8)
- net MCU_G100: now also U403.28 (PA4); no longer U403.37 (PE7)
Changed lines of the file:
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@@
+	)
+	(no_connect
+		(at 144.78 69.85)
 	)
 	(no_connect
@@
 	)
 	(no_connect
-		(at 187.96 44.45)
-	)
-	(no_connect
 		(at 187.96 107.95)
 	)
 	(no_connect
+		(at 144.78 77.47)
+	)
+	(no_connect
 		(at 144.78 118.11)
 	)
@@
 	)
 	(no_connect
-		(at 187.96 41.91)
-	)
-	(no_connect
 		(at 187.96 138.43)
 	)
@@
 	)
 	(no_connect
-		(at 187.96 39.37)
-	)
-	(no_connect
 		(at 30.48 41.91)
 	)
 	(no_connect
+		(at 144.78 72.39)
+	)
+	(no_connect
 		(at 187.96 151.13)
 	)
@@
 	(wire
 		(pts
-			(xy 140.97 77.47) (xy 144.78 77.47)
+			(xy 189.23 44.45) (xy 187.96 44.45)
 		)
 		(stroke
@@
 	(wire
 		(pts
-			(xy 140.97 72.39) (xy 144.78 72.39)
+			(xy 189.23 41.91) (xy 187.96 41.91)
 		)
 		(stroke
@@
 	(wire
 		(pts
-			(xy 140.97 69.85) (xy 144.78 69.85)
+			(xy 189.23 39.37) (xy 187.96 39.37)
 		)
 		(stroke
@@
 	(hierarchical_label "MCU_G1"
 		(shape output)
-		(at 140.97 77.47 180)
-		(fields_autoplaced yes)
-		(effects
-			(font
-				(size 1.27 1.27)
-			)
-			(justify right)
+		(at 189.23 44.45 0)
+		(fields_autoplaced yes)
+		(effects
+			(font
+				(size 1.27 1.27)
+			)
+			(justify left)
 		)
 	)
@@
 	(hierarchical_label "MCU_G10"
 		(shape output)
-		(at 140.97 72.39 180)
-		(fields_autoplaced yes)
-		(effects
-			(font
-				(size 1.27 1.27)
-			)
-			(justify right)
+		(at 189.23 41.91 0)
+		(fields_autoplaced yes)
+		(effects
+			(font
+				(size 1.27 1.27)
+			)
+			(justify left)
 		)
 	)
@@
 	(hierarchical_label "MCU_G100"
 		(shape output)
-		(at 140.97 69.85 180)
-		(fields_autoplaced yes)
-		(effects
-			(font
-				(size 1.27 1.27)
-			)
-			(justify right)
-		)
-	)
+		(at 189.23 39.37 0)
+		(fields_autoplaced yes)
+		(effects
+			(font
+				(size 1.27 1.27)
+			)
+			(justify left)
+		)
+	)

Commit message: Development
Parts:
- R201: now not fitted
- U202: footprint Package_TO_SOT_SMD:TSOT-23-5_HandSoldering -> Package_TO_SOT_SMD:TSOT-23-5
Changed lines of the file:
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@@
 			)
 		)
-		(property "Footprint" "Package_TO_SOT_SMD:TSOT-23-5_HandSoldering"
+		(property "Footprint" "Package_TO_SOT_SMD:TSOT-23-5"
 			(at 58.42 134.62 0)
 			(effects
@@
 		(in_bom yes)
 		(on_board yes)
-		(dnp no)
+		(dnp yes)
 		(property "Reference" "R201"
 			(at 58.42 66.294 90)

Commit message: Development
Parts:
- D401: value ASCB-JTC2-0A308 -> ASMB-MTB1-0B3A2
- RN401: value 680 -> EXB-V8V102JV
Changed lines of the file:
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@@
 		(on_board yes)
 		(dnp no)
-		(fields_autoplaced yes)
 		(property "Reference" "D401"
-			(at 46.99 22.86 90)
+			(at 48.006 23.368 90)
 			(effects
 				(font
@@
 			)
 		)
-		(property "Value" "ASCB-JTC2-0A308"
-			(at 54.61 25.4 90)
+		(property "Value" "ASMB-MTB1-0B3A2"
+			(at 55.88 25.908 90)
 			(effects
 				(font
@@
 		(fields_autoplaced yes)
 		(property "Reference" "RN401"
-			(at 33.02 35.56 0)
+			(at 33.02 35.5599 0)
 			(effects
 				(font
@@
 			)
 		)
-		(property "Value" "680"
-			(at 33.02 38.1 0)
+		(property "Value" "EXB-V8V102JV"
+			(at 33.02 38.0999 0)
 			(effects
 				(font

Commit message: PCB design changes.
Parts:
- added C213: DNP, Capacitor_SMD:C_0603_1608Metric_Pad1.08x0.95mm_HandSolder, symbol Device:C
- renumbered R207 to R203, R208 to R204
Connections:
- net +3.3V: no longer C410.1, U201.3 (V+), U201.7 (~{SHDN})
- net +3.3VADC: now also C410.1, U201.3 (V+), U201.7 (~{SHDN})
- net at R201.2, R203.1, U201.1 (-IN1)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: now also C213.1
- net at R204.1, U201.5 (OUT2): now also C213.2
Other:
- moved on the sheet: C410, R201, R203, R204

Commit message: Hardware design
Parts:
- U202: footprint Package_TO_SOT_SMD:TSOT-23-5 -> Package_TO_SOT_SMD:SOT-23-5_HandSoldering
Changed lines of the file:
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@@
 			)
 		)
-		(property "Footprint" "Package_TO_SOT_SMD:TSOT-23-5"
+		(property "Footprint" "Package_TO_SOT_SMD:SOT-23-5_HandSoldering"
 			(at 58.42 134.62 0)
 			(effects
