File: HARDWARE/ETH1ACPL-C79x/Power.kicad_sch (KiCad schematic)
At the start: 18 parts, among them J201 1715721, Q201 SI5618A, Q202 MMBT3904, U201 TSR_1-2450, U202 TLV62568DBV

Commit message: PCB design changes.
Parts:
- removed C204: 10u, Capacitor_SMD:C_1206_3216Metric_Pad1.33x1.80mm_HandSolder, symbol Device:C
- removed C205: 22u, Capacitor_Tantalum_SMD:CP_EIA-3528-21_Kemet-B_Pad1.50x2.35mm_HandSolder, symbol Device:C_Polarized
- removed L201: CSHB0415-2R2M, ETH1ACPL-C79x:CSHB0415, symbol Device:L
- removed R203: 45k3, Resistor_SMD:R_0603_1608Metric_Pad0.98x0.95mm_HandSolder, symbol Device:R
- removed R204: 10k, Resistor_SMD:R_0603_1608Metric_Pad0.98x0.95mm_HandSolder, symbol Device:R
- removed U202: TLV62568DBV, Package_TO_SOT_SMD:SOT-23-5, symbol Regulator_Switching:TLV62568DBV
- added C304: 10u, Capacitor_SMD:C_1206_3216Metric_Pad1.33x1.80mm_HandSolder, symbol Device:C
- added C305: 22u, Capacitor_Tantalum_SMD:CP_EIA-3528-21_Kemet-B_Pad1.50x2.35mm_HandSolder, symbol Device:C_Polarized
- added U302: LM1117MP-3.3/NOPB, Package_TO_SOT_SMD:SOT-223-3_TabPin2, symbol Regulator_Linear:LM1117MP-3.3
Connections:
- net +3.3V: now also C305.1, U302.2 (VO)
- net +5V: now also C304.1, U302.3 (VI)
- net GND: now also C304.2, C305.2, U302.1 (GND)
