File: HARDWARE/ETH1ACPL-C79x/Voltage.kicad_sch (KiCad schematic)
At the start: 60 parts, among them J501 1710072, U501 OPA340UA, U502 TBA 1-0511HI, U504 ACPL-C79B, U505 DG412LEDQ, U506 DG419LEDY, U507 DG412LEDQ, U509 OPA340UA, U510 OPA340UA

Commit message: Development
Parts:
- removed C519, C520, C521: 0.1u, Capacitor_SMD:C_0603_1608Metric_Pad1.08x0.95mm_HandSolder, symbol Device:C
- removed R527: RT1206BRE07900KL, Resistor_SMD:R_1206_3216Metric_Pad1.30x1.75mm_HandSolder, symbol Device:R
- removed RN501: SOT-DIV23LF-03-9002-1002-DD, Package_TO_SOT_SMD:SOT-23, symbol Device:VoltageDivider_CenterPin3
- removed U501, U509, U510: OPA340UA, Package_SO:SOIC-8_3.9x4.9mm_P1.27mm, symbol Amplifier_Operational:OPA340UA
- removed U505: DG412LEDQ, Package_SO:TSSOP-16_4.4x5mm_P0.65mm, symbol Analog_Switch:DG412xUE
- added R518: 100k, Resistor_SMD:R_0603_1608Metric_Pad0.98x0.95mm_HandSolder, symbol Device:R
- added R525: 100k/0.1%, Resistor_SMD:R_0603_1608Metric_Pad0.98x0.95mm_HandSolder, symbol Device:R
- added U505: OPA2340UA, Package_SO:SOIC-8_3.9x4.9mm_P1.27mm, symbol Amplifier_Operational:OPA2340
- R522: value 10k/0.1% -> 6k2/0.1%
- R523: renamed from R521; value 10k/0.1% -> 6k2/0.1%
- U502: footprint (none) -> ETH1ACPL-C79x:TBA1
- renumbered C512 to C501, C515 to C502, C501 to C503, C502 to C504, C518 to C505, C511 to C506, C514 to C507, C507 to C508, C503 to C509, C504 to C510, C517 to C511, C506 to C512, C505 to C513, C508 to C514, C509 to C515, C510 to C516, C525 to C517, R505 to R501, R501 to R502, R509 to R503, R510 to R504, R506 to R505, R502 to R506, R511 to R507, R512 to R508, R507 to R509, R503 to R510, R513 to R511, R514 to R512, R508 to R513, R504 to R514, R518 to R519, R519 to R520, R520 to R521, R528 to R524, R531 to R526, R532 to R527, R533 to R528, R534 to R529, R535 to R530, U507 to U501, U504 to U503, U506 to U504
Connections:
- net +1.65V: now also R529.2, R525.2
- net +3.3V: now also R518.2, U505.8 (V+)
- net GND: now also U505.4 (V-); no longer R529.2
- net at R520.2, R522.2: now also U505.3 (+)
- net at D501.3 (K), R526.2, R527.1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: now also U505.7
- net at R521.2, R523.1: now also U505.2 (-)
- net at R523.2, U504.2: now also U505.1
- net at R526.1: now also U504.1, R525.1, U505.5 (+); no longer U501.14
- net at U501.15: now also U501.14; no longer U504.1
- net at U501.10, U501.2, U501.6: now also U505.6 (-)
- net MCU_MEAS_ENA: no longer names the net of U501.16
- net MCU_MEAS_ENA: now also R518.1
Other:
- moved on the sheet: C501, C502, C503, C504, C505, C506, C507, C508, C509, C510, C511, C512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

Commit message: Development
Parts:
- C509, C510, C517, R519, R526: now not fitted
- R530: value 100 -> 0
Other:
- note added: "56k = ERA-8VRB5602V"
Changed lines of the file:
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@@
 	)
 	(junction
-		(at 257.81 86.36)
+		(at 261.62 86.36)
 		(diameter 0)
 		(color 0 0 0 0)
@@
 	(wire
 		(pts
-			(xy 257.81 86.36) (xy 261.62 86.36)
+			(xy 261.62 86.36) (xy 265.43 86.36)
 		)
 		(stroke
@@
 	(wire
 		(pts
+			(xy 256.54 86.36) (xy 261.62 86.36)
+		)
+		(stroke
+			(width 0)
+			(type default)
+		)
+	)
+	(wire
+		(pts
 			(xy 160.02 39.37) (xy 160.02 38.1)
 		)
@@
 	(wire
 		(pts
-			(xy 256.54 86.36) (xy 257.81 86.36)
-		)
-		(stroke
-			(width 0)
-			(type default)
-		)
-	)
-	(wire
-		(pts
 			(xy 36.83 90.17) (xy 36.83 91.44)
 		)
@@
 		)
 	)
+	(text "56k = ERA-8VRB5602V"
+		(exclude_from_sim no)
+		(at 57.912 109.474 0)
+		(effects
+			(font
+				(size 1.27 1.27)
+			)
+		)
+	)
 	(hierarchical_label "VOUT"
 		(shape output)
-		(at 261.62 86.36 0)
+		(at 265.43 86.36 0)
 		(fields_autoplaced yes)
 		(effects
@@
 		(in_bom yes)
 		(on_board yes)
-		(dnp no)
+		(dnp yes)
 		(fields_autoplaced yes)
 		(property "Reference" "C509"
@@
 	(symbol
 		(lib_id "Device:C")
-		(at 257.81 90.17 0)
+		(at 261.62 90.17 0)
 		(unit 1)
 		(exclude_from_sim no)
 		(in_bom yes)
 		(on_board yes)
-		(dnp no)
+		(dnp yes)
 		(fields_autoplaced yes)
 		(property "Reference" "C517"
-			(at 260.985 89.535 0)
+			(at 264.795 89.535 0)
 			(effects
 				(font
@@
 		)
 		(property "Value" "100p"
-			(at 260.985 92.075 0)
+			(at 264.795 92.075 0)
 			(effects
 				(font
@@
 		)
 		(property "Footprint" "Capacitor_SMD:C_0603_1608Metric_Pad1.08x0.95mm_HandSolder"
-			(at 258.7752 93.98 0)
+			(at 262.5852 93.98 0)
 			(effects
 				(font
@@
 		)
 		(property "Datasheet" "~"
-			(at 257.81 90.17 0)
+			(at 261.62 90.17 0)
 			(effects
 				(font
@@
 		)
 		(property "Description" ""
-			(at 257.81 90.17 0)
+			(at 261.62 90.17 0)
 			(effects
 				(font
@@
 		(in_bom yes)
 		(on_board yes)
-		(dnp no)
+		(dnp yes)
 		(fields_autoplaced yes)
 		(property "Reference" "R526"
@@
 			)
 		)
-		(property "Value" "100"
+		(property "Value" "0"
 			(at 252.73 83.82 90)
 			(effects
@@
 	(symbol
 		(lib_id "power:GND")
-		(at 257.81 93.98 0)
+		(at 261.62 93.98 0)
 		(unit 1)
 		(exclude_from_sim no)
@@
 		(dnp no)
 		(property "Reference" "#PWR0528"
-			(at 257.81 100.33 0)
+			(at 261.62 100.33 0)
 			(effects
 				(font
@@
 		)
 		(property "Value" "GND"
-			(at 257.81 98.425 0)
+			(at 261.62 98.425 0)
 			(effects
 				(font
@@
 		)
 		(property "Footprint" ""
-			(at 257.81 93.98 0)
+			(at 261.62 93.98 0)
 			(effects
 				(font
@@
 		)
 		(property "Datasheet" ""
-			(at 257.81 93.98 0)
+			(at 261.62 93.98 0)
 			(effects
 				(font
@@
 		)
 		(property "Description" "Power symbol creates a global label with name \"GND\" , ground"
-			(at 257.81 93.98 0)
+			(at 261.62 93.98 0)
 			(effects
 				(font
@@
 		(in_bom yes)
 		(on_board yes)
-		(dnp no)
+		(dnp yes)
 		(fields_autoplaced yes)
 		(property "Reference" "R519"
@@
 		(in_bom yes)
 		(on_board yes)
-		(dnp no)
+		(dnp yes)
 		(fields_autoplaced yes)
 		(property "Reference" "C510"

Commit message: Development
Other:
- note added: "56k = ERA-8VRB5602V 56 = ERA-3VEB56R0V"
- note removed: "56k = ERA-8VRB5602V"
Changed lines of the file:
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@@
-	)
-	(junction
-		(at 36.83 91.44)
-		(diameter 0)
-		(color 0 0 0 0)
 	)
 	(junction
@@
 	)
 	(junction
-		(at 36.83 71.12)
-		(diameter 0)
-		(color 0 0 0 0)
-	)
-	(junction
 		(at 77.47 180.34)
 		(diameter 0)
@@
 	(wire
 		(pts
-			(xy 33.02 91.44) (xy 33.02 82.55)
+			(xy 33.02 95.25) (xy 33.02 82.55)
 		)
 		(stroke
@@
 	(wire
 		(pts
-			(xy 36.83 91.44) (xy 36.83 95.25)
-		)
-		(stroke
-			(width 0)
-			(type default)
-		)
-	)
-	(wire
-		(pts
 			(xy 77.47 95.25) (xy 93.98 95.25)
 		)
@@
 	(wire
 		(pts
-			(xy 36.83 71.12) (xy 36.83 72.39)
-		)
-		(stroke
-			(width 0)
-			(type default)
-		)
-	)
-	(wire
-		(pts
 			(xy 147.32 38.1) (xy 134.62 38.1)
 		)
@@
 	(wire
 		(pts
-			(xy 33.02 71.12) (xy 36.83 71.12)
+			(xy 33.02 66.04) (xy 36.83 66.04)
 		)
 		(stroke
@@
 	(wire
 		(pts
-			(xy 33.02 71.12) (xy 33.02 80.01)
+			(xy 33.02 66.04) (xy 33.02 80.01)
 		)
 		(stroke
@@
 	(wire
 		(pts
-			(xy 36.83 90.17) (xy 36.83 91.44)
+			(xy 36.83 90.17) (xy 36.83 95.25)
 		)
 		(stroke
@@
 	(wire
 		(pts
-			(xy 33.02 91.44) (xy 36.83 91.44)
+			(xy 33.02 95.25) (xy 36.83 95.25)
 		)
 		(stroke
@@
 	(wire
 		(pts
-			(xy 36.83 66.04) (xy 36.83 71.12)
+			(xy 36.83 66.04) (xy 36.83 72.39)
 		)
 		(stroke
@@
 		)
 	)
-	(text "56k = ERA-8VRB5602V"
+	(text "56k = ERA-8VRB5602V\n56 = ERA-3VEB56R0V"
 		(exclude_from_sim no)
 		(at 57.912 109.474 0)

Commit message: Development
Parts:
- added SYM501, SYM502: SYM_Flash_Small, ETH1ACPL-C79x:Symbol_Attention_Triangle_8x7mm_Copper, symbol Graphic:SYM_Flash_Small
Connections:
- net +1.65V: now also R524.2
- net GND: no longer R524.2
Changed lines of the file:
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@@
+	)
+	(symbol
+		(lib_id "ETH1ACPL-C79x:+1.65V")
+		(at 170.18 95.25 180)
+		(unit 1)
+		(exclude_from_sim no)
+		(in_bom yes)
+		(on_board yes)
+		(dnp no)
+		(property "Reference" "#PWR0524"
+			(at 166.37 93.98 0)
+			(effects
+				(font
+					(size 1.27 1.27)
+				)
+				(hide yes)
+			)
+		)
+		(property "Value" "+1.65V"
+			(at 170.18 99.06 0)
+			(effects
+				(font
+					(size 1.27 1.27)
+				)
+			)
+		)
+		(property "Footprint" ""
+			(at 170.18 95.25 0)
+			(effects
+				(font
+					(size 1.27 1.27)
+				)
+				(hide yes)
+			)
+		)
+		(property "Datasheet" ""
+			(at 170.18 95.25 0)
+			(effects
+				(font
+					(size 1.27 1.27)
+				)
+				(hide yes)
+			)
+		)
+		(property "Description" "Power symbol creates a global label with name \"+1.65V\""
+			(at 170.18 95.25 0)
+			(effects
+				(font
+					(size 1.27 1.27)
+				)
+				(hide yes)
+			)
+		)
+		(pin "1"
+		)
+		(instances
+			(project "ETH1ACPL-C79x"
+				(path "/e8a00664-7a76-490e-9471-410cd41c5487/0c5ac836-56da-45d2-a861-346d6ac8e804"
+					(reference "#PWR0524")
+					(unit 1)
+				)
+			)
+		)
 	)
 	(symbol
@@
 	)
 	(symbol
+		(lib_id "Graphic:SYM_Flash_Small")
+		(at 31.75 30.48 0)
+		(unit 1)
+		(exclude_from_sim yes)
+		(in_bom no)
+		(on_board yes)
+		(dnp no)
+		(fields_autoplaced yes)
+		(property "Reference" "SYM502"
+			(at 29.464 30.48 90)
+			(effects
+				(font
+					(size 1.27 1.27)
+				)
+				(hide yes)
+			)
+		)
+		(property "Value" "SYM_Flash_Small"
+			(at 34.036 30.48 90)
+			(effects
+				(font
+					(size 1.27 1.27)
+				)
+				(hide yes)
+			)
+		)
+		(property "Footprint" "ETH1ACPL-C79x:Symbol_Attention_Triangle_8x7mm_Copper"
+			(at 31.75 31.115 0)
+			(effects
+				(font
+					(size 1.27 1.27)
+				)
+				(hide yes)
+			)
+		)
+		(property "Datasheet" "~"
+			(at 41.91 33.02 0)
+			(effects
+				(font
+					(size 1.27 1.27)
+				)
+				(hide yes)
+			)
+		)
+		(property "Description" "Flash symbol, small"
+			(at 31.75 30.48 0)
+			(effects
+				(font
+					(size 1.27 1.27)
+				)
+				(hide yes)
+			)
+		)
+		(instances
+			(project "ETH1ACPL-C79x"
+				(path "/e8a00664-7a76-490e-9471-410cd41c5487/0c5ac836-56da-45d2-a861-346d6ac8e804"
+					(reference "SYM502")
+					(unit 1)
+				)
+			)
+		)
+	)
+	(symbol
 		(lib_id "Device:R")
 		(at 72.39 66.04 90)
@@
 				(path "/e8a00664-7a76-490e-9471-410cd41c5487/0c5ac836-56da-45d2-a861-346d6ac8e804"
 					(reference "R514")
-					(unit 1)
-				)
-			)
-		)
-	)
-	(symbol
-		(lib_id "power:GND")
-		(at 170.18 95.25 0)
-		(unit 1)
-		(exclude_from_sim no)
-		(in_bom yes)
-		(on_board yes)
-		(dnp no)
-		(property "Reference" "#PWR0524"
-			(at 170.18 101.6 0)
-			(effects
-				(font
-					(size 1.27 1.27)
-				)
-				(hide yes)
-			)
-		)
-		(property "Value" "GND"
-			(at 170.18 99.314 0)
-			(effects
-				(font
-					(size 1.27 1.27)
-				)
-			)
-		)
-		(property "Footprint" ""
-			(at 170.18 95.25 0)
-			(effects
-				(font
-					(size 1.27 1.27)
-				)
-				(hide yes)
-			)
-		)
-		(property "Datasheet" ""
-			(at 170.18 95.25 0)
-			(effects
-				(font
-					(size 1.27 1.27)
-				)
-				(hide yes)
-			)
-		)
-		(property "Description" "Power symbol creates a global label with name \"GND\" , ground"
-			(at 170.18 95.25 0)
-			(effects
-				(font
-					(size 1.27 1.27)
-				)
-				(hide yes)
-			)
-		)
-		(pin "1"
-		)
-		(instances
-			(project "ETH1ACPL-C79x"
-				(path "/e8a00664-7a76-490e-9471-410cd41c5487/0c5ac836-56da-45d2-a861-346d6ac8e804"
-					(reference "#PWR0524")
 					(unit 1)
 				)
@@
 					(unit 1)
 				)
+			)
+		)
+	)
+	(symbol
+		(lib_id "Graphic:SYM_Flash_Small")
+		(at 22.86 30.48 0)
+		(unit 1)
+		(exclude_from_sim no)
+		(in_bom no)
+		(on_board yes)
+		(dnp no)
+		(fields_autoplaced yes)
+		(property "Reference" "SYM501"
+			(at 20.574 30.48 90)
+			(effects
+				(font
+					(size 1.27 1.27)
+				)
+				(hide yes)
+			)
+		)
+		(property "Value" "SYM_Flash_Small"
+			(at 25.146 30.48 90)
+			(effects
+				(font
+					(size 1.27 1.27)
+				)
+				(hide yes)
+			)
+		)
+		(property "Footprint" "ETH1ACPL-C79x:Symbol_Attention_Triangle_8x7mm_Copper"
+			(at 22.86 31.115 0)
+			(effects
+				(font
+					(size 1.27 1.27)
+				)
+				(hide yes)
+			)
+		)
+		(property "Datasheet" "~"
+			(at 33.02 33.02 0)
+			(effects
+				(font
+					(size 1.27 1.27)
+				)
+				(hide yes)
+			)
+		)
+		(property "Description" "Flash symbol, small"
+			(at 22.86 30.48 0)
+			(effects
+				(font
+					(size 1.27 1.27)
+				)
+				(hide yes)
+			)
+		)
+		(property "Sim.Enable" "0"
+			(at 22.86 30.48 0)
+			(effects
+				(font
+					(size 1.27 1.27)
+				)
+				(hide yes)
+			)
+		)
+		(instances
+			(project "ETH1ACPL-C79x"
+				(path "/e8a00664-7a76-490e-9471-410cd41c5487/0c5ac836-56da-45d2-a861-346d6ac8e804"
+					(reference "SYM501")
+					(unit 1)
+				)

Commit message: PCB design changes.
Parts:
- removed R526: 0, Resistor_SMD:R_0603_1608Metric_Pad0.98x0.95mm_HandSolder, symbol Device:R
- R526: renamed from R527; value 180k/0.1% -> 180k/0.05%
- R527: renamed from R528; value 18k/0.1% -> 18k/0.05%
- R528: renamed from R529; value 2k/0.1% -> 2k/0.05%
- renumbered R530 to R529, U504 to U502, U502 to U503, U503 to U504
Other:
- moved on the sheet: D501

Commit message: Hardware design
Parts:
- added C518, C519: 68p, Capacitor_SMD:C_0603_1608Metric_Pad1.08x0.95mm_HandSolder, symbol Device:C
- added RN501, RN502: MPMT50011002AT5, Package_TO_SOT_SMD:SOT-23, symbol Device:VoltageDivider_CenterPin3
Connections:
- net +1.65V: now also C519.2, RN501.1
- net at R520.2, R522.2, U505.3 (+): now also C519.1, RN501.3
- net at R521.2, R523.1, U505.2 (-): now also C518.1, RN502.3
- net at R523.2, U502.2, U505.1: now also C518.2, RN502.1
- net at R520.1, U504.7 (OUT+): now also RN501.2
- net at R521.1, U504.6 (OUT-): now also RN502.2
Other:
- moved on the sheet: C517, D501, R522, R523, R524, R525, R526, R527, R528, R529, U501A, U501B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
